File: LT/Integration/Mobo_Rev1/29_4NotchFilter.sch (KiCad schematic (older format))
At the start: 24 parts

Commit message: STEP files
I attempted to add as many step files into the Mother Board kicad as I could
Parts:
- C40, C41, C42, C43, C44, C45, C46, C47: footprint (none) -> LT:CAP_Trimmer_TZB4Z
Changed lines of the file:
@@
 EESchema Schematic File Version 4
-EELAYER 30 0
+LIBS:Mobo_Rev1-cache
+EELAYER 26 0
 EELAYER END
 $Descr A4 11693 8268
@@
 F 0 "C40" H 6415 1746 50  0000 L CNN
 F 1 "C_Variable" H 6415 1655 50  0000 L CNN
-F 2 "" H 6300 1700 50  0001 C CNN
+F 2 "LT:CAP_Trimmer_TZB4Z" H 6300 1700 50  0001 C CNN
 F 3 "~" H 6300 1700 50  0001 C CNN
 	1    6300 1700
@@
 F 0 "C41" H 6415 2196 50  0000 L CNN
 F 1 "C_Variable" H 6415 2105 50  0000 L CNN
-F 2 "" H 6300 2150 50  0001 C CNN
+F 2 "LT:CAP_Trimmer_TZB4Z" H 6300 2150 50  0001 C CNN
 F 3 "~" H 6300 2150 50  0001 C CNN
 	1    6300 2150
@@
 F 0 "C42" H 7065 1746 50  0000 L CNN
 F 1 "C_Variable" H 7065 1655 50  0000 L CNN
-F 2 "" H 6950 1700 50  0001 C CNN
+F 2 "LT:CAP_Trimmer_TZB4Z" H 6950 1700 50  0001 C CNN
 F 3 "~" H 6950 1700 50  0001 C CNN
 	1    6950 1700
@@
 F 0 "C43" H 7065 2196 50  0000 L CNN
 F 1 "C_Variable" H 7065 2105 50  0000 L CNN
-F 2 "" H 6950 2150 50  0001 C CNN
+F 2 "LT:CAP_Trimmer_TZB4Z" H 6950 2150 50  0001 C CNN
 F 3 "~" H 6950 2150 50  0001 C CNN
 	1    6950 2150
@@
 F 0 "C44" H 7765 1746 50  0000 L CNN
 F 1 "C_Variable" H 7765 1655 50  0000 L CNN
-F 2 "" H 7650 1700 50  0001 C CNN
+F 2 "LT:CAP_Trimmer_TZB4Z" H 7650 1700 50  0001 C CNN
 F 3 "~" H 7650 1700 50  0001 C CNN
 	1    7650 1700
@@
 F 0 "C45" H 7765 2196 50  0000 L CNN
 F 1 "C_Variable" H 7765 2105 50  0000 L CNN
-F 2 "" H 7650 2150 50  0001 C CNN
+F 2 "LT:CAP_Trimmer_TZB4Z" H 7650 2150 50  0001 C CNN
 F 3 "~" H 7650 2150 50  0001 C CNN
 	1    7650 2150
@@
 F 0 "C46" H 8415 1746 50  0000 L CNN
 F 1 "C_Variable" H 8415 1655 50  0000 L CNN
-F 2 "" H 8300 1700 50  0001 C CNN
+F 2 "LT:CAP_Trimmer_TZB4Z" H 8300 1700 50  0001 C CNN
 F 3 "~" H 8300 1700 50  0001 C CNN
 	1    8300 1700
@@
 F 0 "C47" H 8415 2196 50  0000 L CNN
 F 1 "C_Variable" H 8415 2105 50  0000 L CNN
-F 2 "" H 8300 2150 50  0001 C CNN
+F 2 "LT:CAP_Trimmer_TZB4Z" H 8300 2150 50  0001 C CNN
 F 3 "~" H 8300 2150 50  0001 C CNN
 	1    8300 2150

Commit message: Just a push check
idk if I pushed
Parts:
- C40, C41, C42, C43, C44, C45, C46, C47: footprint LT:CAP_Trimmer_TZB4Z -> LT:CAP_trimmer_SGC3_Download
Changed lines of the file:
@@
 F 0 "C40" H 6415 1746 50  0000 L CNN
 F 1 "C_Variable" H 6415 1655 50  0000 L CNN
-F 2 "LT:CAP_Trimmer_TZB4Z" H 6300 1700 50  0001 C CNN
+F 2 "LT:CAP_trimmer_SGC3_Download" H 6300 1700 50  0001 C CNN
 F 3 "~" H 6300 1700 50  0001 C CNN
 	1    6300 1700
@@
 F 0 "C41" H 6415 2196 50  0000 L CNN
 F 1 "C_Variable" H 6415 2105 50  0000 L CNN
-F 2 "LT:CAP_Trimmer_TZB4Z" H 6300 2150 50  0001 C CNN
+F 2 "LT:CAP_trimmer_SGC3_Download" H 6300 2150 50  0001 C CNN
 F 3 "~" H 6300 2150 50  0001 C CNN
 	1    6300 2150
@@
 F 0 "C42" H 7065 1746 50  0000 L CNN
 F 1 "C_Variable" H 7065 1655 50  0000 L CNN
-F 2 "LT:CAP_Trimmer_TZB4Z" H 6950 1700 50  0001 C CNN
+F 2 "LT:CAP_trimmer_SGC3_Download" H 6950 1700 50  0001 C CNN
 F 3 "~" H 6950 1700 50  0001 C CNN
 	1    6950 1700
@@
 F 0 "C43" H 7065 2196 50  0000 L CNN
 F 1 "C_Variable" H 7065 2105 50  0000 L CNN
-F 2 "LT:CAP_Trimmer_TZB4Z" H 6950 2150 50  0001 C CNN
+F 2 "LT:CAP_trimmer_SGC3_Download" H 6950 2150 50  0001 C CNN
 F 3 "~" H 6950 2150 50  0001 C CNN
 	1    6950 2150
@@
 F 0 "C44" H 7765 1746 50  0000 L CNN
 F 1 "C_Variable" H 7765 1655 50  0000 L CNN
-F 2 "LT:CAP_Trimmer_TZB4Z" H 7650 1700 50  0001 C CNN
+F 2 "LT:CAP_trimmer_SGC3_Download" H 7650 1700 50  0001 C CNN
 F 3 "~" H 7650 1700 50  0001 C CNN
 	1    7650 1700
@@
 F 0 "C45" H 7765 2196 50  0000 L CNN
 F 1 "C_Variable" H 7765 2105 50  0000 L CNN
-F 2 "LT:CAP_Trimmer_TZB4Z" H 7650 2150 50  0001 C CNN
+F 2 "LT:CAP_trimmer_SGC3_Download" H 7650 2150 50  0001 C CNN
 F 3 "~" H 7650 2150 50  0001 C CNN
 	1    7650 2150
@@
 F 0 "C46" H 8415 1746 50  0000 L CNN
 F 1 "C_Variable" H 8415 1655 50  0000 L CNN
-F 2 "LT:CAP_Trimmer_TZB4Z" H 8300 1700 50  0001 C CNN
+F 2 "LT:CAP_trimmer_SGC3_Download" H 8300 1700 50  0001 C CNN
 F 3 "~" H 8300 1700 50  0001 C CNN
 	1    8300 1700
@@
 F 0 "C47" H 8415 2196 50  0000 L CNN
 F 1 "C_Variable" H 8415 2105 50  0000 L CNN
-F 2 "LT:CAP_Trimmer_TZB4Z" H 8300 2150 50  0001 C CNN
+F 2 "LT:CAP_trimmer_SGC3_Download" H 8300 2150 50  0001 C CNN
 F 3 "~" H 8300 2150 50  0001 C CNN
 	1    8300 2150
