File: LT/Integration/Mobo_Rev1/PreAmp.sch (KiCad schematic (older format))
At the start: 8 parts, among them Q2 5486

Commit message: STEP files
I attempted to add as many step files into the Mother Board kicad as I could
Parts:
- C4, C5: footprint LT:CAP_trimmer_SGC3 -> LT:CAP_trimmer_SGC3_Download
Changed lines of the file:
@@
 EESchema Schematic File Version 4
-EELAYER 30 0
+LIBS:Mobo_Rev1-cache
+EELAYER 26 0
 EELAYER END
 $Descr A4 11693 8268
@@
 F 0 "C4" H 3365 1996 50  0000 L CNN
 F 1 "SGC3" H 3365 1905 50  0000 L CNN
-F 2 "LT:CAP_trimmer_SGC3" H 3250 1950 50  0001 C CNN
+F 2 "LT:CAP_trimmer_SGC3_Download" H 3250 1950 50  0001 C CNN
 F 3 "~" H 3250 1950 50  0001 C CNN
 	1    3250 1950
@@
 F 0 "C5" H 4015 1996 50  0000 L CNN
 F 1 "SGC3" H 4015 1905 50  0000 L CNN
-F 2 "LT:CAP_trimmer_SGC3" H 3900 1950 50  0001 C CNN
+F 2 "LT:CAP_trimmer_SGC3_Download" H 3900 1950 50  0001 C CNN
 F 3 "~" H 3900 1950 50  0001 C CNN
 	1    3900 1950
