File: LT/Integration/Dobo_Rev1/IF.sch (KiCad schematic (older format))
At the start: 16 parts, among them Y1 Crystal_GND2, Y2 Crystal_GND2

Commit message: Daughter Board
Began annotating the rest of the Daughter board
Parts:
- L11, L12, L13, L14: footprint (none) -> Inductor_SMD:L_0805_2012Metric
- R27, R28: footprint (none) -> Resistor_SMD:R_0805_2012Metric
Changed lines of the file:
@@
 F 0 "R27" H 5170 3546 50  0000 L CNN
 F 1 "R" H 5170 3455 50  0000 L CNN
-F 2 "" V 5030 3500 50  0001 C CNN
+F 2 "Resistor_SMD:R_0805_2012Metric" V 5030 3500 50  0001 C CNN
 F 3 "~" H 5100 3500 50  0001 C CNN
 	1    5100 3500
@@
 F 0 "R28" H 5420 3546 50  0000 L CNN
 F 1 "R" H 5420 3455 50  0000 L CNN
-F 2 "" V 5280 3500 50  0001 C CNN
+F 2 "Resistor_SMD:R_0805_2012Metric" V 5280 3500 50  0001 C CNN
 F 3 "~" H 5350 3500 50  0001 C CNN
 	1    5350 3500
@@
 F 0 "L11" H 5953 3346 50  0000 L CNN
 F 1 "L" H 5953 3255 50  0000 L CNN
-F 2 "" H 5900 3300 50  0001 C CNN
+F 2 "Inductor_SMD:L_0805_2012Metric" H 5900 3300 50  0001 C CNN
 F 3 "~" H 5900 3300 50  0001 C CNN
 	1    5900 3300
@@
 F 0 "L12" H 6103 3346 50  0000 L CNN
 F 1 "L" H 6103 3255 50  0000 L CNN
-F 2 "" H 6050 3300 50  0001 C CNN
+F 2 "Inductor_SMD:L_0805_2012Metric" H 6050 3300 50  0001 C CNN
 F 3 "~" H 6050 3300 50  0001 C CNN
 	1    6050 3300
@@
 F 0 "L13" H 6303 3346 50  0000 L CNN
 F 1 "L" H 6303 3255 50  0000 L CNN
-F 2 "" H 6250 3300 50  0001 C CNN
+F 2 "Inductor_SMD:L_0805_2012Metric" H 6250 3300 50  0001 C CNN
 F 3 "~" H 6250 3300 50  0001 C CNN
 	1    6250 3300
@@
 F 0 "L14" H 6503 3346 50  0000 L CNN
 F 1 "L" H 6503 3255 50  0000 L CNN
-F 2 "" H 6450 3300 50  0001 C CNN
+F 2 "Inductor_SMD:L_0805_2012Metric" H 6450 3300 50  0001 C CNN
 F 3 "~" H 6450 3300 50  0001 C CNN
 	1    6450 3300

Commit message: Finished Daughter Board
I finished assigning the footprints to the daughter board
Parts:
- Y1, Y2: footprint (none) -> Crystal:Crystal_HC49-U-3Pin_Vertical
Changed lines of the file:
@@
 F 0 "Y1" H 7400 4168 50  0000 C CNN
 F 1 "Crystal_GND2" H 7400 4077 50  0000 C CNN
-F 2 "" H 7400 3900 50  0001 C CNN
+F 2 "Crystal:Crystal_HC49-U-3Pin_Vertical" H 7400 3900 50  0001 C CNN
 F 3 "~" H 7400 3900 50  0001 C CNN
 	1    7400 3900
@@
 F 0 "Y2" H 7900 4168 50  0000 C CNN
 F 1 "Crystal_GND2" H 7900 4077 50  0000 C CNN
-F 2 "" H 7900 3900 50  0001 C CNN
+F 2 "Crystal:Crystal_HC49-U-3Pin_Vertical" H 7900 3900 50  0001 C CNN
 F 3 "~" H 7900 3900 50  0001 C CNN
 	1    7900 3900

Commit message: Messing With Resistors
Just doing some resistor changes but idk if it worked
Parts:
- R27, R28: symbol Device:R -> Dobo_Rev1-rescue:R-Device
Changed lines of the file:
@@
 $EndComp
 $Comp
-L Device:R R27
+L Dobo_Rev1-rescue:R-Device R27
 U 1 1 5E4C0C18
 P 5100 3500
@@
 $EndComp
 $Comp
-L Device:R R28
+L Dobo_Rev1-rescue:R-Device R28
 U 1 1 5E4C135E
 P 5350 3500
