File: LT/Mixer/Down Mixer/Rev1/Down_Mixer_Rev1.sch (KiCad schematic (older format))
At the start: 15 parts

Commit message: updated down-mixer revisions. created a new Rev0.1 for off-the-shelf transformers
Parts:
- removed C? (x2): 10u, symbol Device:C
- removed J?: Conn_Coaxial, symbol Connector:Conn_Coaxial
- removed T?: 3:16, symbol Device:Transformer_1P_1S
- removed T?: 8:1, symbol Device:Transformer_1P_1S
- added C1: 24p, Capacitor_SMD:C_0805_2012Metric_Pad1.15x1.40mm_HandSolder, symbol Device:C
- added C7, C8: 10u, Capacitor_SMD:C_0805_2012Metric_Pad1.15x1.40mm_HandSolder, symbol Device:C
- added C9: 56p, Capacitor_SMD:C_0805_2012Metric_Pad1.15x1.40mm_HandSolder, symbol Device:C
- added J3: Conn_Coaxial, Connector_Coaxial:SMA_Amphenol_132289_EdgeMount, symbol Connector:Conn_Coaxial
- added J4: Conn_01x02_Male, Connector_PinHeader_2.54mm:PinHeader_1x02_P2.54mm_Vertical, symbol Connector:Conn_01x02_Male
- added L1: 2uH, Inductor_SMD:L_0805_2012Metric_Pad1.15x1.40mm_HandSolder, symbol Device:L
- added L3: 3.9u, Inductor_SMD:L_0805_2012Metric_Pad1.15x1.40mm_HandSolder, symbol Device:L
- C2, C3, C4, C5, C6: renamed from C?; footprint (none) -> Capacitor_SMD:C_0805_2012Metric_Pad1.15x1.40mm_HandSolder
- J1, J2: renamed from J?; footprint (none) -> Connector_Coaxial:SMA_Amphenol_132289_EdgeMount
- L2, L4: renamed from L?; footprint (none) -> Inductor_SMD:L_0805_2012Metric_Pad1.15x1.40mm_HandSolder
- U1: renamed from U?; footprint (none) -> Package_SO:SO-8_3.9x4.9mm_P1.27mm; symbol LT-Schematics:SA602 -> Down_Mixer_Rev2-rescue:SA602-LT-Schematics
Connections:
- net GND: now also C3.2, C1.2, C8.2, C9.2, J3.2 (Ext), J4.1 (Pin_1)
- net VCC: now also J4.2 (Pin_2)
- net at U1.4 (OUT_A): now also C8.1
- net at U1.5 (OUT_B): now also C7.1
- net at C2.2: now also L1.2
- net at J1.1 (In): now also C1.1, L1.1
- new net: C7.2, L3.2
- new net: C9.1, J3.1 (In), L3.1

Commit message: completed down-mixer rev0.1 schematic and layout. generated milling files
Parts:
- U1: symbol Down_Mixer_Rev2-rescue:SA602-LT-Schematics -> Down_Mixer_Rev1-rescue:SA602-LT-Schematics-Down_Mixer_Rev2-rescue
Changed lines of the file:
@@
 $EndComp
 $Comp
-L Down_Mixer_Rev2-rescue:SA602-LT-Schematics U1
+L Down_Mixer_Rev1-rescue:SA602-LT-Schematics-Down_Mixer_Rev2-rescue U1
 U 1 1 5E447907
 P 5000 3750
