File: LT/Local-Oscillator/Rev-4/Rev 4.02/PLL Board Rev4.02.sch (KiCad schematic (older format))
At the start: 69 parts, among them J1 Conn_01x02_Male, J13 Conn_01x02_Male, J14 Conn_01x02_Male, J15 Conn_01x02_Male, J16 Conn_01x02_Male, J17 Conn_01x02_Male, J18 Conn_Coaxial, J2 Conn_Coaxial, J20 Conn_01x02_Male, J3 Conn_Coaxial, J4 Conn_01x04_Male, J5 Conn_01x02_Male, J7 Conn_01x02_Male, J8 Conn_01x02_Male, Q1 2N5486 JFET, Q2 2N5486 JFET, U1 LMX231X, U2 L7808

Commit message: Imported Rev4.01, 4.02, 4.03 to Kicad
Put Rev4.01, Rev4.02, and Rev4.03 onto KiCad
Parts:
- removed U1: LMX231X, LMX231X:LMX231X, symbol Complete-PLL-Board-Rev4-rescue:LMX231X-LMX2313
- added U1: LMX231X, LT:LMX231X, symbol LMX2313:LMX231X
- D3, D4: value 1SV232 -> ???
- R1, R10, R11, R12, R2, R3, R4, R5, R6, R7, R8, R9: symbol Device:R -> PLL-Board-Rev4.02-rescue:R-Device-Complete-PLL-Board-Rev4-rescue-PLL-Board-Rev4.01-rescue
- R13, R14: value 1k -> 0k; symbol Device:R -> PLL-Board-Rev4.02-rescue:R-Device-Complete-PLL-Board-Rev4-rescue-PLL-Board-Rev4.01-rescue
Other:
- note added: "1/3/20"
- note added: "Rev4.02: Unknown Varactor Values"
- note removed: "3/3/19"
Changed lines of the file:
@@
 EESchema Schematic File Version 4
-LIBS:Complete PLL Board Rev4-cache
-EELAYER 26 0
+EELAYER 30 0
 EELAYER END
 $Descr A4 11693 8268
@@
 $EndComp
 $Comp
-L Device:R R1
+L PLL-Board-Rev4.02-rescue:R-Device-Complete-PLL-Board-Rev4-rescue-PLL-Board-Rev4.01-rescue R1
 U 1 1 5C6B70C1
 P 2500 1400
@@
 $EndComp
 $Comp
-L Device:R R3
+L PLL-Board-Rev4.02-rescue:R-Device-Complete-PLL-Board-Rev4-rescue-PLL-Board-Rev4.01-rescue R3
 U 1 1 5C6B724B
 P 3500 1350
@@
 $EndComp
 $Comp
-L Device:R R4
+L PLL-Board-Rev4.02-rescue:R-Device-Complete-PLL-Board-Rev4-rescue-PLL-Board-Rev4.01-rescue R4
 U 1 1 5C6B7281
 P 4000 1350
@@
 	2450 3250 4150 3250
 $Comp
-L Device:R R2
+L PLL-Board-Rev4.02-rescue:R-Device-Complete-PLL-Board-Rev4-rescue-PLL-Board-Rev4.01-rescue R2
 U 1 1 5C6B86E4
 P 2800 2100
@@
 P 6750 4700
 F 0 "D3" V 6750 4900 50  0000 R CNN
-F 1 "1SV232" V 6650 5050 50  0000 R CNN
+F 1 "???" V 6650 5050 50  0000 R CNN
 F 2 "Diode_SMD:D_SC-80_HandSoldering" H 6750 4700 50  0001 C CNN
 F 3 "~" H 6750 4700 50  0001 C CNN
@@
 P 6750 5250
 F 0 "D4" V 6750 5350 50  0000 L CNN
-F 1 "1SV232" V 6850 5300 50  0000 L CNN
+F 1 "???" V 6850 5300 50  0000 L CNN
 F 2 "Diode_SMD:D_SC-80_HandSoldering" H 6750 5250 50  0001 C CNN
 F 3 "~" H 6750 5250 50  0001 C CNN
@@
 $EndComp
 $Comp
-L Device:R R9
+L PLL-Board-Rev4.02-rescue:R-Device-Complete-PLL-Board-Rev4-rescue-PLL-Board-Rev4.01-rescue R9
 U 1 1 5C802100
 P 8800 5200
@@
 	8100 5050 8100 5150
 $Comp
-L Device:R R10
+L PLL-Board-Rev4.02-rescue:R-Device-Complete-PLL-Board-Rev4-rescue-PLL-Board-Rev4.01-rescue R10
 U 1 1 5C809914
 P 9600 5050
@@
 $EndComp
 $Comp
-L Device:R R11
+L PLL-Board-Rev4.02-rescue:R-Device-Complete-PLL-Board-Rev4-rescue-PLL-Board-Rev4.01-rescue R11
 U 1 1 5C80AB36
 P 9950 5500
@@
 PLL Board
 Text Notes 8150 7650 0    50   Italic 10
-3/3/19
+1/3/20
 Text Notes 10600 7650 0    50   ~ 10
 1
-$Comp
-L Complete-PLL-Board-Rev4-rescue:LMX231X-LMX2313 U1
-U 1 1 5C7E02DA
-P 4850 2300
-F 0 "U1" H 4700 1550 50  0000 C CNN
-F 1 "LMX231X" H 4700 1450 50  0000 C CNN
-F 2 "LMX231X:LMX231X" H 4350 2000 50  0001 C CNN
-F 3 "" H 4350 2000 50  0001 C CNN
-	1    4850 2300
-	1    0    0    -1
-$EndComp
 Text GLabel 9050 3000 1    50   Input ~ 0
 8V
@@
 Connection ~ 7200 1850
 $Comp
-L Device:R R6
+L PLL-Board-Rev4.02-rescue:R-Device-Complete-PLL-Board-Rev4-rescue-PLL-Board-Rev4.01-rescue R6
 U 1 1 5C863D30
 P 7700 1850
@@
 	7800 3000 7900 3000
 $Comp
-L Device:R R5
+L PLL-Board-Rev4.02-rescue:R-Device-Complete-PLL-Board-Rev4-rescue-PLL-Board-Rev4.01-rescue R5
 U 1 1 5C8FC8A8
 P 7500 2850
@@
 	8800 4750 8800 4900
 $Comp
-L Device:R R8
+L PLL-Board-Rev4.02-rescue:R-Device-Complete-PLL-Board-Rev4-rescue-PLL-Board-Rev4.01-rescue R8
 U 1 1 5CA66BF5
 P 9400 4900
@@
 $EndComp
 $Comp
-L Device:R R7
+L PLL-Board-Rev4.02-rescue:R-Device-Complete-PLL-Board-Rev4-rescue-PLL-Board-Rev4.01-rescue R7
 U 1 1 5CA7D1B6
 P 7550 1300
@@
 Connection ~ 9950 4550
 $Comp
-L Device:R R12
+L PLL-Board-Rev4.02-rescue:R-Device-Complete-PLL-Board-Rev4-rescue-PLL-Board-Rev4.01-rescue R12
 U 1 1 5CB9DB4B
 P 6500 5100
@@
 	8800 4900 8950 4900
 $Comp
-L Device:R R13
+L PLL-Board-Rev4.02-rescue:R-Device-Complete-PLL-Board-Rev4-rescue-PLL-Board-Rev4.01-rescue R13
 U 1 1 5CBB0D39
 P 6150 4400
 F 0 "R13" V 6350 4350 50  0000 L CNN
-F 1 "1k" V 6250 4350 50  0000 L CNN
+F 1 "0k" V 6250 4350 50  0000 L CNN
 F 2 "Resistor_SMD:R_0805_2012Metric_Pad1.15x1.40mm_HandSolder" V 6080 4400 50  0001 C CNN
 F 3 "~" H 6150 4400 50  0001 C CNN
@@
 $EndComp
 $Comp
-L Device:R R14
+L PLL-Board-Rev4.02-rescue:R-Device-Complete-PLL-Board-Rev4-rescue-PLL-Board-Rev4.01-rescue R14
 U 1 1 5CBBAAF0
 P 6300 4400
 F 0 "R14" V 6500 4350 50  0000 L CNN
-F 1 "1k" V 6400 4350 50  0000 L CNN
+F 1 "0k" V 6400 4350 50  0000 L CNN
 F 2 "Resistor_SMD:R_0805_2012Metric_Pad1.15x1.40mm_HandSolder" V 6230 4400 50  0001 C CNN
 F 3 "~" H 6300 4400 50  0001 C CNN
@@
 Wire Wire Line
 	7950 1850 8350 1850
+$Comp
+L LMX2313:LMX231X U1
+U 1 1 5E5B770A
+P 4850 2300
+F 0 "U1" H 4700 1500 50  0000 C CNN
+F 1 "LMX231X" H 4750 1400 50  0000 C CNN
+F 2 "LT:LMX231X" H 4350 2000 50  0001 C CNN
+F 3 "" H 4350 2000 50  0001 C CNN
+	1    4850 2300
+	1    0    0    -1
+$EndComp
+Text Notes 2350 7150 0    79   ~ 16
+Rev4.02: Unknown Varactor Values
 $EndSCHEMATC
