File: LT/Power-Amplifier/PA 2020/PA Rev 4.0/PA Rev 4.0.sch (KiCad schematic (older format))
At the start: 16 parts, among them J0 Power, J1 RF IN, J2 RF OUT, T1 RF XFormer, T2 RF Xformer

Commit message: PA Rev 4.0 layout is complete. PCB is ready to be milled
Parts:
- J1, J2: footprint Connector_Coaxial:SMA_Molex_73251-1153_EdgeMount_Horizontal -> PA:SMAConnector
Changed lines of the file:
@@
 F 0 "J1" H 856 3928 50  0000 C CNN
 F 1 "RF IN" H 856 3837 50  0000 C CNN
-F 2 "Connector_Coaxial:SMA_Molex_73251-1153_EdgeMount_Horizontal" H 750 3750 50  0001 C CNN
+F 2 "PA:SMAConnector" H 750 3750 50  0001 C CNN
 F 3 "~" H 750 3750 50  0001 C CNN
 	1    750  3750
@@
 F 0 "J2" H 5756 3928 50  0000 C CNN
 F 1 "RF OUT" H 5756 3837 50  0000 C CNN
-F 2 "Connector_Coaxial:SMA_Molex_73251-1153_EdgeMount_Horizontal" H 5650 3750 50  0001 C CNN
+F 2 "PA:SMAConnector" H 5650 3750 50  0001 C CNN
 F 3 "~" H 5650 3750 50  0001 C CNN
 	1    5650 3750
