File: SE/Flash_Memory_Interface/Flash_Memory_Interface.sch (KiCad schematic (older format))
At the start: 5 parts

Commit message: Finished SE Flash Memory Schematic
Parts:
- removed J?: Conn_01x06_Male, symbol Connector:Conn_01x06_Male
- removed J?: Conn_01x03_Male, symbol Connector:Conn_01x03_Male
- removed U?: SN74LVC2G04DBVR, DBV6, symbol 2020-03-08_23-19-55:SN74LVC2G04DBVR
- added J?: Conn_01x06_Male, symbol Connector:Conn_01x06_Male
- added J? (x2): Conn_01x02_Male, symbol Connector:Conn_01x02_Male
- added J?: Conn_01x01_Male, symbol Connector:Conn_01x01_Male
- added U?: SN74LVC32APWR, PW14, symbol SE-Schematics:SN74LVC32APWR
- added U?: SN74LVC2G04DBVR, DBV6, symbol SE-Schematics:SN74LVC2G04DBVR
- added U? (x6): 74AHCV541A, symbol SE-Schematics:74AHCV541A
- added U? (x2): MT29F2G08AABWP, symbol flash_memory:MT29F2G08AABWP
Connections:
- net labels added: +3.3V, ChipSelect, CombinationalLogic1, CombinationalLogic2, CombinationalLogic3, CombinationalLogic4, CombinationalLogic5, Flash_ControlBus_0, Flash_ControlBus_1, Flash_ControlBus_2, Flash_ControlBus_3, Flash_ControlBus_4, Flash_ControlBus_5, Flash_ControlBus_6, GND, IO_0, IO_1, IO_2, IO_3, IO_4, IO_5, IO_6, IO_7, MicroController_ControlBus_0, MicroController_ControlBus_1, MicroController_ControlBus_2, MicroController_ControlBus_3, MicroController_ControlBus_4, MicroController_ControlBus_5, MicroController_R_B_Interrupt, ReadWrite, Vcc
- wire segments 0 -> 165
- no-connect marks 0 -> 8
Other:
- note added: "Chip Select\n"
- note added: "Control Bus\nMicrocontroller"
- note added: "I/O\nMicrocontroller"
- note added: "MicroController\n R/B Interrupt"
- note added: "Read/Write"
- note removed: "Control Bus [5:0]"
- note removed: "I/O from Microcontroller"
- moved on the sheet: J?, U?

Commit message: Changed an input pin to the flash memory for SE schematic
Parts:
- U?: symbol SE-Schematics:SN74LVC32APWR -> Flash_Memory_Interface-rescue:SN74LVC32APWR-SE-Schematics
- U?: symbol SE-Schematics:SN74LVC2G04DBVR -> Flash_Memory_Interface-rescue:SN74LVC2G04DBVR-SE-Schematics
- U? (x6): symbol SE-Schematics:74AHCV541A -> Flash_Memory_Interface-rescue:74AHCV541A-SE-Schematics
- U? (x2): symbol flash_memory:MT29F2G08AABWP -> Flash_Memory_Interface-rescue:MT29F2G08AABWP-flash_memory
Connections:
- net Flash_ControlBus_2: no longer U?.10 (CE2), U?.10 (CE2)
- new net: U?.11 (Y7), U?.11 (Y7) (x2)
- new net: U?.13 (Y5), U?.15 (Y3) (x2)
- no-connect marks 8 -> 10
Other:
- note added: "3"
- note added: "Flash Memory Scheme v.3"
- moved on the sheet: J?, U?
