File: LT/Integration/Mobo_Rev0/29_4NotchFilter.sch (KiCad schematic (older format))
At the start: 24 parts

Commit message: Annotating components for Transmitting stage. In progress
Parts:
- renumbered C34 to C46, C35 to C47, C36 to C48, C37 to C49, C38 to C51, C39 to C52, C40 to C53, C41 to C54, C42 to C55, C43 to C56, C44 to C57, C45 to C58, C46 to C59, C47 to C60
Changed lines of the file:
@@
 $EndComp
 $Comp
-L Device:C C34
+L Device:C C46
 U 1 1 5E4C4B72
 P 3100 1700
-F 0 "C34" H 3215 1746 50  0000 L CNN
+F 0 "C46" H 3215 1746 50  0000 L CNN
 F 1 "C" H 3215 1655 50  0000 L CNN
 F 2 "" H 3138 1550 50  0001 C CNN
@@
 $EndComp
 $Comp
-L Device:C C36
+L Device:C C48
 U 1 1 5E4C4C25
 P 3400 1700
-F 0 "C36" H 3515 1746 50  0000 L CNN
+F 0 "C48" H 3515 1746 50  0000 L CNN
 F 1 "C" H 3515 1655 50  0000 L CNN
 F 2 "" H 3438 1550 50  0001 C CNN
@@
 $EndComp
 $Comp
-L Device:C C38
+L Device:C C51
 U 1 1 5E4C4C7A
 P 3750 1700
-F 0 "C38" H 3865 1746 50  0000 L CNN
+F 0 "C51" H 3865 1746 50  0000 L CNN
 F 1 "C" H 3865 1655 50  0000 L CNN
 F 2 "" H 3788 1550 50  0001 C CNN
@@
 $EndComp
 $Comp
-L Device:C C35
+L Device:C C47
 U 1 1 5E4C4D12
 P 3100 2150
-F 0 "C35" H 3215 2196 50  0000 L CNN
+F 0 "C47" H 3215 2196 50  0000 L CNN
 F 1 "C" H 3215 2105 50  0000 L CNN
 F 2 "" H 3138 2000 50  0001 C CNN
@@
 $EndComp
 $Comp
-L Device:C C37
+L Device:C C49
 U 1 1 5E4C4D19
 P 3400 2150
-F 0 "C37" H 3515 2196 50  0000 L CNN
+F 0 "C49" H 3515 2196 50  0000 L CNN
 F 1 "C" H 3515 2105 50  0000 L CNN
 F 2 "" H 3438 2000 50  0001 C CNN
@@
 $EndComp
 $Comp
-L Device:C C39
+L Device:C C52
 U 1 1 5E4C4D20
 P 3750 2150
-F 0 "C39" H 3865 2196 50  0000 L CNN
+F 0 "C52" H 3865 2196 50  0000 L CNN
 F 1 "C" H 3865 2105 50  0000 L CNN
 F 2 "" H 3788 2000 50  0001 C CNN
@@
 $EndComp
 $Comp
-L Device:C_Variable C40
+L Device:C_Variable C53
 U 1 1 5E4C4E32
 P 6300 1700
-F 0 "C40" H 6415 1746 50  0000 L CNN
+F 0 "C53" H 6415 1746 50  0000 L CNN
 F 1 "C_Variable" H 6415 1655 50  0000 L CNN
 F 2 "" H 6300 1700 50  0001 C CNN
@@
 $EndComp
 $Comp
-L Device:C_Variable C41
+L Device:C_Variable C54
 U 1 1 5E4C4ECB
 P 6300 2150
-F 0 "C41" H 6415 2196 50  0000 L CNN
+F 0 "C54" H 6415 2196 50  0000 L CNN
 F 1 "C_Variable" H 6415 2105 50  0000 L CNN
 F 2 "" H 6300 2150 50  0001 C CNN
@@
 $EndComp
 $Comp
-L Device:C_Variable C42
+L Device:C_Variable C55
 U 1 1 5E4C4F33
 P 6950 1700
-F 0 "C42" H 7065 1746 50  0000 L CNN
+F 0 "C55" H 7065 1746 50  0000 L CNN
 F 1 "C_Variable" H 7065 1655 50  0000 L CNN
 F 2 "" H 6950 1700 50  0001 C CNN
@@
 $EndComp
 $Comp
-L Device:C_Variable C43
+L Device:C_Variable C56
 U 1 1 5E4C4FA4
 P 6950 2150
-F 0 "C43" H 7065 2196 50  0000 L CNN
+F 0 "C56" H 7065 2196 50  0000 L CNN
 F 1 "C_Variable" H 7065 2105 50  0000 L CNN
 F 2 "" H 6950 2150 50  0001 C CNN
@@
 $EndComp
 $Comp
-L Device:C_Variable C44
+L Device:C_Variable C57
 U 1 1 5E4C5012
 P 7650 1700
-F 0 "C44" H 7765 1746 50  0000 L CNN
+F 0 "C57" H 7765 1746 50  0000 L CNN
 F 1 "C_Variable" H 7765 1655 50  0000 L CNN
 F 2 "" H 7650 1700 50  0001 C CNN
@@
 $EndComp
 $Comp
-L Device:C_Variable C45
+L Device:C_Variable C58
 U 1 1 5E4C5082
 P 7650 2150
-F 0 "C45" H 7765 2196 50  0000 L CNN
+F 0 "C58" H 7765 2196 50  0000 L CNN
 F 1 "C_Variable" H 7765 2105 50  0000 L CNN
 F 2 "" H 7650 2150 50  0001 C CNN
@@
 $EndComp
 $Comp
-L Device:C_Variable C46
+L Device:C_Variable C59
 U 1 1 5E4C5115
 P 8300 1700
-F 0 "C46" H 8415 1746 50  0000 L CNN
+F 0 "C59" H 8415 1746 50  0000 L CNN
 F 1 "C_Variable" H 8415 1655 50  0000 L CNN
 F 2 "" H 8300 1700 50  0001 C CNN
@@
 $EndComp
 $Comp
-L Device:C_Variable C47
+L Device:C_Variable C60
 U 1 1 5E4C511C
 P 8300 2150
-F 0 "C47" H 8415 2196 50  0000 L CNN
+F 0 "C60" H 8415 2196 50  0000 L CNN
 F 1 "C_Variable" H 8415 2105 50  0000 L CNN
 F 2 "" H 8300 2150 50  0001 C CNN

Commit message: Working on Transmitting Stage rev 0 integration board. Still in progress
Parts:
- C46, C47, C48, C49, C51: footprint (none) -> Capacitor_SMD:C_0805_2012Metric_Pad1.15x1.40mm_HandSolder
Changed lines of the file:
@@
 F 0 "C46" H 3215 1746 50  0000 L CNN
 F 1 "C" H 3215 1655 50  0000 L CNN
-F 2 "" H 3138 1550 50  0001 C CNN
+F 2 "Capacitor_SMD:C_0805_2012Metric_Pad1.15x1.40mm_HandSolder" H 3138 1550 50  0001 C CNN
 F 3 "~" H 3100 1700 50  0001 C CNN
 	1    3100 1700
@@
 F 0 "C48" H 3515 1746 50  0000 L CNN
 F 1 "C" H 3515 1655 50  0000 L CNN
-F 2 "" H 3438 1550 50  0001 C CNN
+F 2 "Capacitor_SMD:C_0805_2012Metric_Pad1.15x1.40mm_HandSolder" H 3438 1550 50  0001 C CNN
 F 3 "~" H 3400 1700 50  0001 C CNN
 	1    3400 1700
@@
 F 0 "C51" H 3865 1746 50  0000 L CNN
 F 1 "C" H 3865 1655 50  0000 L CNN
-F 2 "" H 3788 1550 50  0001 C CNN
+F 2 "Capacitor_SMD:C_0805_2012Metric_Pad1.15x1.40mm_HandSolder" H 3788 1550 50  0001 C CNN
 F 3 "~" H 3750 1700 50  0001 C CNN
 	1    3750 1700
@@
 F 0 "C47" H 3215 2196 50  0000 L CNN
 F 1 "C" H 3215 2105 50  0000 L CNN
-F 2 "" H 3138 2000 50  0001 C CNN
+F 2 "Capacitor_SMD:C_0805_2012Metric_Pad1.15x1.40mm_HandSolder" H 3138 2000 50  0001 C CNN
 F 3 "~" H 3100 2150 50  0001 C CNN
 	1    3100 2150
@@
 F 0 "C49" H 3515 2196 50  0000 L CNN
 F 1 "C" H 3515 2105 50  0000 L CNN
-F 2 "" H 3438 2000 50  0001 C CNN
+F 2 "Capacitor_SMD:C_0805_2012Metric_Pad1.15x1.40mm_HandSolder" H 3438 2000 50  0001 C CNN
 F 3 "~" H 3400 2150 50  0001 C CNN
 	1    3400 2150
