File: LT/Integration/Mobo_Rev1/Mobo_Dev1/VA.sch (KiCad schematic (older format))
At the start: 0 parts

Commit message: Adding the files for the phase 2 receiving stage for LT Integration
Parts:
- added C1, C2: 220pF, Capacitor_SMD:C_0402_1005Metric, symbol Device:C
- added C10, C11, C8, C9: 10nF, Capacitor_SMD:C_0402_1005Metric, symbol Device:C
- added C3, C4: 22pF, Capacitor_SMD:C_0402_1005Metric, symbol Device:C
- added C5, C6: 330pF, Capacitor_SMD:C_0402_1005Metric, symbol Device:C
- added C7: 10nH, Capacitor_SMD:C_0402_1005Metric, symbol Device:C
- added J2: Conn_Coaxial, Connector_Coaxial:SMA_Amphenol_132289_EdgeMount, symbol Connector:Conn_Coaxial
- added J3, J4: Conn_01x02_Male, Connector_PinHeader_2.54mm:PinHeader_1x02_P2.54mm_Vertical, symbol Connector:Conn_01x02_Male
- added L1, L2: 3.9nH, Inductor_SMD:L_0402_1005Metric, symbol Device:L
- added L3, L4, L5, L6: 47nH, Inductor_SMD:L_0402_1005Metric, symbol Device:L
- added L7, L8: 150nH, Inductor_SMD:L_0402_1005Metric, symbol Device:L
- added R1, R2: 120, Resistor_SMD:R_0402_1005Metric, symbol Device:R_US
- added R3, R4: 330, Resistor_SMD:R_0402_1005Metric, symbol Device:R_US
- added U1: BAP64Q, LT:BAP64Q, symbol LT-Schematics:BAP64Q
Connections:
- new net: C2.1, C4.1, C6.1, J2.1 (In), L2.2
- new net: L2.1, L3.1, L6.1
- new net: L3.2, L6.2, L8.1
- new net: C9.2, L8.2
- new net: C9.1, R4.2, U1.1 (I/O)
- new net: R1.1, R2.1, U1.2
- new net: C8.1, R3.1, U1.3 (I/O2)
- new net: L1.1, L4.1, L5.1
- new net: L4.2, L5.2, L7.1
- new net: C7.1, J3.1 (Pin_1), R1.2, R2.2
- new net: C8.2, L7.2
- new net +5V: C10.1, C11.1, J4.1 (Pin_1), U1.4 (PWR1), U1.5 (PWR2)
- new net GND: C1.2, C10.2, C11.2, C2.2, C3.2, C4.2, C5.2, C6.2, C7.2, J2.2 (Ext), J3.2 (Pin_2), J4.2 (Pin_2), R3.2, R4.1
- new net Variable_Attenuator_Out: C1.1, C3.1, C5.1, L1.2
Other:
- note added: "Control Voltage (Vr)"
- note added: "RF in"
- note added: "RF out"
- note added: "from Pre-select"
- note added: "to LNA"
