File: LT/Integration/Mobo_Phase3/PreAmp.sch (KiCad schematic (older format))
At the start: 0 parts

Commit message: Finished schematic layout of Pre Amplifier
Parts:
- added C30: C_Variable, LT:CAP_trimmer_SGC3_Download, symbol Device:C_Variable
- added C31, C32: 1uF, Capacitor_SMD:C_0402_1005Metric, symbol Daisy~Chain-cache:Device_C
- added J8: Conn_01x02_Male, Connector_PinHeader_2.54mm:PinHeader_1x02_P2.54mm_Vertical, symbol Connector:Conn_01x02_Male
- added J9: Conn_01x02_Female, Connector_PinSocket_2.54mm:PinSocket_1x02_P2.54mm_Vertical, symbol Connector:Conn_01x02_Female
- added L22, L23: LTRIM, LT:IND_trimmer_7M3, symbol Device:LTRIM
- added Q2: Q_NJFET_DSG, Package_TO_SOT_SMD:SOT-23, symbol Device:Q_NJFET_DSG
- added R12: 0, Resistor_SMD:R_0805_2012Metric_Pad1.15x1.40mm_HandSolder, symbol Device:R
Connections:
- new net: C30.2, R12.1
- new net: C31.1, J8.1 (Pin_1), L23.1
- new net: C30.1, L22.1, Q2.3 (G)
- new net: C32.2, L23.2, Q2.1 (D)
- new net: C32.1, J9.1 (Pin_1)
- new net 29.4BPF_OUT: R12.2
- new net GND: C31.2, J8.2 (Pin_2), J9.2 (Pin_2), L22.2, Q2.2 (S)
Changed lines of the file:
@@
 EESchema Schematic File Version 4
-EELAYER 30 0
+LIBS:Mobo_Phase3-cache
+EELAYER 26 0
 EELAYER END
 $Descr A4 11693 8268
 encoding utf-8
-Sheet 1 8
+Sheet 6 8
 Title ""
 Date ""
@@
 Comment4 ""
 $EndDescr
+$Comp
+L Device:R R12
+U 1 1 5EB62A6B
+P 3200 3150
+F 0 "R12" V 2993 3150 50  0000 C CNN
+F 1 "0" V 3084 3150 50  0000 C CNN
+F 2 "Resistor_SMD:R_0805_2012Metric_Pad1.15x1.40mm_HandSolder" V 3130 3150 50  0001 C CNN
+F 3 "~" H 3200 3150 50  0001 C CNN
+	1    3200 3150
+	0    1    1    0
+$EndComp
+$Comp
+L Daisy~Chain-cache:Device_C C31
+U 1 1 5EB62BDE
+P 4350 2500
+F 0 "C31" H 4100 2550 50  0000 L CNN
+F 1 "1uF" H 4100 2450 50  0000 L CNN
+F 2 "Capacitor_SMD:C_0402_1005Metric" H 4388 2350 50  0001 C CNN
+F 3 "" H 4350 2500 50  0001 C CNN
+	1    4350 2500
+	1    0    0    -1
+$EndComp
+Text HLabel 2800 3150 0    50   Input ~ 0
+29.4BPF_OUT
+Wire Wire Line
+	2800 3150 3050 3150
+$Comp
+L Device:C_Variable C30
+U 1 1 5EB63DB3
+P 3700 3150
+F 0 "C30" V 3448 3150 50  0000 C CNN
+F 1 "C_Variable" V 3539 3150 50  0000 C CNN
+F 2 "LT:CAP_trimmer_SGC3_Download" H 3700 3150 50  0001 C CNN
+F 3 "~" H 3700 3150 50  0001 C CNN
+	1    3700 3150
+	0    1    1    0
+$EndComp
+Wire Wire Line
+	3350 3150 3550 3150
+$Comp
+L Device:LTRIM L22
+U 1 1 5EB63EB5
+P 4000 3300
+F 0 "L22" H 4102 3346 50  0000 L CNN
+F 1 "LTRIM" H 4102 3255 50  0000 L CNN
+F 2 "LT:IND_trimmer_7M3" H 4000 3300 50  0001 C CNN
+F 3 "~" H 4000 3300 50  0001 C CNN
+	1    4000 3300
+	1    0    0    -1
+$EndComp
+$Comp
+L power:GND #PWR0104
+U 1 1 5EB63F78
+P 4000 3450
+F 0 "#PWR0104" H 4000 3200 50  0001 C CNN
+F 1 "GND" H 4005 3277 50  0000 C CNN
+F 2 "" H 4000 3450 50  0001 C CNN
+F 3 "" H 4000 3450 50  0001 C CNN
+	1    4000 3450
+	1    0    0    -1
+$EndComp
+Wire Wire Line
+	4000 3150 3850 3150
+$Comp
+L Device:Q_NJFET_DSG Q2
+U 1 1 5EB64019
+P 4550 3150
+F 0 "Q2" H 4741 3196 50  0000 L CNN
+F 1 "Q_NJFET_DSG" H 4741 3105 50  0000 L CNN
+F 2 "Package_TO_SOT_SMD:SOT-23" H 4750 3250 50  0001 C CNN
+F 3 "~" H 4550 3150 50  0001 C CNN
+	1    4550 3150
+	1    0    0    -1
+$EndComp
+Wire Wire Line
+	4350 3150 4000 3150
+Connection ~ 4000 3150
+$Comp
+L power:GND #PWR0105
+U 1 1 5EB640D0
+P 4650 3350
+F 0 "#PWR0105" H 4650 3100 50  0001 C CNN
+F 1 "GND" H 4655 3177 50  0000 C CNN
+F 2 "" H 4650 3350 50  0001 C CNN
+F 3 "" H 4650 3350 50  0001 C CNN
+	1    4650 3350
+	1    0    0    -1
+$EndComp
+$Comp
+L Device:LTRIM L23
+U 1 1 5EB640E5
+P 4650 2500
+F 0 "L23" H 4752 2546 50  0000 L CNN
+F 1 "LTRIM" H 4752 2455 50  0000 L CNN
+F 2 "LT:IND_trimmer_7M3" H 4650 2500 50  0001 C CNN
+F 3 "~" H 4650 2500 50  0001 C CNN
+	1    4650 2500
+	1    0    0    -1
+$EndComp
+Wire Wire Line
+	4650 2650 4650 2850
+Wire Wire Line
+	4350 2350 4650 2350
+$Comp
+L power:GND #PWR0106
+U 1 1 5EB64270
+P 4350 2650
+F 0 "#PWR0106" H 4350 2400 50  0001 C CNN
+F 1 "GND" H 4355 2477 50  0000 C CNN
+F 2 "" H 4350 2650 50  0001 C CNN
+F 3 "" H 4350 2650 50  0001 C CNN
+	1    4350 2650
+	1    0    0    -1
+$EndComp
+$Comp
+L Connector:Conn_01x02_Male J8
+U 1 1 5EB64300
+P 4650 1950
+F 0 "J8" V 4710 1763 50  0000 R CNN
+F 1 "Conn_01x02_Male" V 4801 1763 50  0000 R CNN
+F 2 "Connector_PinHeader_2.54mm:PinHeader_1x02_P2.54mm_Vertical" H 4650 1950 50  0001 C CNN
+F 3 "~" H 4650 1950 50  0001 C CNN
+	1    4650 1950
+	0    -1   1    0
+$EndComp
+Wire Wire Line
+	4650 2150 4650 2350
+Connection ~ 4650 2350
+$Comp
+L power:GND #PWR0107
+U 1 1 5EB64481
+P 4750 2150
+F 0 "#PWR0107" H 4750 1900 50  0001 C CNN
+F 1 "GND" H 4900 2050 50  0000 C CNN
+F 2 "" H 4750 2150 50  0001 C CNN
+F 3 "" H 4750 2150 50  0001 C CNN
+	1    4750 2150
+	1    0    0    -1
+$EndComp
+$Comp
+L Daisy~Chain-cache:Device_C C32
+U 1 1 5EB6449A
+P 5200 2850
+F 0 "C32" V 5050 2800 50  0000 L CNN
+F 1 "1uF" V 5350 2800 50  0000 L CNN
+F 2 "Capacitor_SMD:C_0402_1005Metric" H 5238 2700 50  0001 C CNN
+F 3 "" H 5200 2850 50  0001 C CNN
+	1    5200 2850
+	0    1    1    0
+$EndComp
+Wire Wire Line
+	5050 2850 4650 2850
+Connection ~ 4650 2850
+Wire Wire Line
+	4650 2850 4650 2950
+$Comp
+L Connector:Conn_01x02_Female J9
+U 1 1 5EB64662
+P 5550 2850
+F 0 "J9" H 5577 2826 50  0000 L CNN
+F 1 "Conn_01x02_Female" H 5577 2735 50  0000 L CNN
+F 2 "Connector_PinSocket_2.54mm:PinSocket_1x02_P2.54mm_Vertical" H 5550 2850 50  0001 C CNN
+F 3 "~" H 5550 2850 50  0001 C CNN
+	1    5550 2850
+	1    0    0    -1
+$EndComp
+$Comp
+L power:GND #PWR0108
+U 1 1 5EB64C4A
+P 5350 2950
+F 0 "#PWR0108" H 5350 2700 50  0001 C CNN
+F 1 "GND" H 5355 2777 50  0000 C CNN
+F 2 "" H 5350 2950 50  0001 C CNN
+F 3 "" H 5350 2950 50  0001 C CNN
+	1    5350 2950
+	1    0    0    -1
+$EndComp
 $EndSCHEMATC
