File: LT/Integration/Final Integration Layouts/Phase 3/DoBo/Dobo_Phase3/Up-Mixer.sch (KiCad schematic (older format))
At the start: 15 parts, among them J5 Conn_Coaxial, T1 Transformer_6, T2 Transformer_6, U2 SA602

Commit message: uploaded the final schematics for the integration
Connections:
- net Up_Mixer_input renamed Up_Mixer_Input
Changed lines of the file:
@@
 $EndComp
 Text HLabel 2500 3850 0    50   Input ~ 0
-Up_Mixer_input
+Up_Mixer_Input
 Wire Wire Line
 	2550 3850 2500 3850
