File: LT/Pre-Amplifier/Pre-Amplifier/Pre-Amplifier.kicad_pcb (KiCad board)
At the start: 2 copper layers, 43.2 x 38.8 mm, 9 parts, among them J1 Conn_Coaxial, J2 Conn_Coaxial, J3 Conn_01x02_Male, Q1 Q_NJFET_DSG

Commit message: Preamplifier KiCad Revisions
Parts:
- added C4: 39pF, Capacitor_SMD:C_0805_2012Metric_Pad1.18x1.45mm_HandSolder, F.Cu at (170.3, 77.6)
- added C5: 220nF, Capacitor_SMD:C_0805_2012Metric_Pad1.18x1.45mm_HandSolder, F.Cu at (133.9, 90.8)
- added C6: 220nF, Capacitor_SMD:C_0805_2012Metric_Pad1.18x1.45mm_HandSolder, F.Cu at (164.3, 106.4)
- added C7: 3.9nF, Capacitor_SMD:C_0805_2012Metric_Pad1.18x1.45mm_HandSolder, F.Cu at (158.1, 90.2)
- added C8: 39pF, Capacitor_SMD:C_0805_2012Metric_Pad1.18x1.45mm_HandSolder, F.Cu at (173.4, 97.5)
- added J4: Conn_01x02_Male, Connector_PinHeader_2.54mm:PinHeader_1x02_P2.54mm_Vertical, F.Cu at (151.3, 103.8)
- added L3: 150uH, Inductor_SMD:L_0805_2012Metric_Pad1.15x1.40mm_HandSolder, F.Cu at (138.3, 81.3)
- added L4: 150uH, Inductor_SMD:L_0805_2012Metric_Pad1.15x1.40mm_HandSolder, F.Cu at (138.9, 93.5)
- added Q2: Q_PNP_BCE, Package_TO_SOT_SMD:SOT-23_Handsoldering, F.Cu at (163.8, 80.5)
- added Q3: Q_PNP_BCE, Package_TO_SOT_SMD:SOT-23_Handsoldering, F.Cu at (148.8, 93.0)
- added Q4: Q_NPN_BCE, Package_TO_SOT_SMD:SOT-23_Handsoldering, F.Cu at (166.1, 97.3)
- added R1: 1.8M, Resistor_SMD:R_0805_2012Metric_Pad1.20x1.40mm_HandSolder, F.Cu at (143.2, 77.1)
- added R2: 20k, Resistor_SMD:R_0805_2012Metric_Pad1.20x1.40mm_HandSolder, F.Cu at (138.2, 73.8)
- added R3: 1, Resistor_SMD:R_0805_2012Metric_Pad1.20x1.40mm_HandSolder, F.Cu at (162.4, 86.1)
- added R4: 1, Resistor_SMD:R_0805_2012Metric_Pad1.20x1.40mm_HandSolder, F.Cu at (159.3, 78.2)
- added R5: 51k, Resistor_SMD:R_0805_2012Metric_Pad1.20x1.40mm_HandSolder, F.Cu at (139.4, 101.2)
- added R6: 1, Resistor_SMD:R_0805_2012Metric_Pad1.20x1.40mm_HandSolder, F.Cu at (162.4, 90.2)
- added R7: 1.8M, Resistor_SMD:R_0805_2012Metric_Pad1.20x1.40mm_HandSolder, F.Cu at (141.6, 97.5)
- added R8: 1, Resistor_SMD:R_0805_2012Metric_Pad1.20x1.40mm_HandSolder, F.Cu at (169.5, 101.5)
- added T1: Transformer_1P_SS, Transformer_SMD:Transformer_MACOM_SM-22, B.Cu at (122.8, 87.9)
- added T2: Transformer_1P_SS, Transformer_SMD:Transformer_MACOM_SM-22, F.Cu at (182.8, 88.4)
- C1: value C_Variable -> 220nF; footprint LT:CAP_trimmer_SGC3_Download -> Capacitor_SMD:C_0805_2012Metric_Pad1.18x1.45mm_HandSolder
- C2: value 1uF -> 3.9nF; footprint Capacitor_SMD:C_0805_2012Metric_Pad1.15x1.40mm_HandSolder -> Capacitor_SMD:C_0805_2012Metric_Pad1.18x1.45mm_HandSolder
- C3: value C -> 220nF; footprint Capacitor_SMD:C_0805_2012Metric_Pad1.15x1.40mm_HandSolder -> Capacitor_SMD:C_0805_2012Metric_Pad1.18x1.45mm_HandSolder
- J1, J2: footprint Connector_Coaxial:SMA_Amphenol_132289_EdgeMount -> Connector_Coaxial:SMA_Molex_73251-1153_EdgeMount_Horizontal
- L1: value LTRIM -> 0.51uH; footprint LT:IND_trimmer_7M3 -> Inductor_SMD:L_0805_2012Metric_Pad1.15x1.40mm_HandSolder
- L2: value 1.8-2.6uH -> 0.51uH; footprint LT:IND_trimmer_7M3 -> Inductor_SMD:L_0805_2012Metric_Pad1.15x1.40mm_HandSolder
- Q1: value Q_NJFET_DSG -> Q_NPN_BCE; footprint Package_TO_SOT_SMD:SOT-23 -> Package_TO_SOT_SMD:SOT-23_Handsoldering
- moved J2 35.2 mm to (201.5, 88.8), turned to 180 degrees
- moved L2 29.0 mm to (168.8, 106.2), turned to 270 degrees
- moved J1 28.9 mm to (112.5, 88.5), turned to 0 degrees
- moved L1 21.9 mm to (165.5, 74.5)
- moved J3 18.3 mm to (150.1, 71.6), turned to 90 degrees
- moved C1 18.1 mm to (134.0, 85.1)
- moved Q1 13.8 mm to (151.6, 82.0)
- moved C3 4.57 mm to (161.3, 74.2), turned to 270 degrees
- moved C2 2.54 mm to (158.1, 86.1), turned to 270 degrees
Connections:
- C2 pad 1: +8V -> Net-(C2-Pad1)
- C3 pad 2: Net-(C3-Pad2) -> GND
- J1 pad 1: Net-(C1-Pad2) -> Net-(J1-Pad1)
- J2 pad 1: Net-(C3-Pad1) -> Net-(J2-Pad1)
- J3 pad 1: +8V -> Net-(C3-Pad1)
- L1 pad 1: GND -> Net-(C3-Pad1)
- L1 pad 2: (no net) -> Net-(C4-Pad2)
- L2 pad 1: +8V -> Net-(C8-Pad2)
- L2 pad 2: (no net) -> Net-(C6-Pad1)
- Q1 pad 1: Net-(C3-Pad2) -> Net-(C1-Pad1)
- Q1 pad 2: GND -> Net-(Q1-Pad2)
- Q1 pad 3: Net-(C1-Pad1) -> Net-(C2-Pad1)
Routing:
- net Net-(C1-Pad1): track 22.7 -> 0.00 mm
- net Net-(C3-Pad2): track 11.2 -> 0.00 mm
- net Net-(C3-Pad1): track 7.89 -> 0.00 mm
- net +8V: track 7.61 -> 0.00 mm
- net Net-(C1-Pad2): track 6.63 -> 0.00 mm
- removed copper zone on B.Cu, net GND
- removed copper zone on F.Cu, net GND
Other:
- board outline removed
